File: hardware/rp27c512.kicad_sch (KiCad schematic)
At the start: 5 parts, among them J1 Conn_01x17, J2 Conn_01x17, J3 Conn_01x04, U1 27C512

Commit message: added comment
Other:
- title: (none) -> RP2040 27C512 Emulation Board
Changed lines of the file:
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@@
 	(generator_version "8.0")
 	(paper "A4")
+	(title_block
+		(title "RP2040 27C512 Emulation Board")
+		(date "2024-10-27")
+		(rev "1.0")
+	)
 	(junction
 		(at 132.08 57.15)
