File: hardware/rp27c512.kicad_sch (KiCad schematic)
At the start: 5 parts, among them J1 Conn_01x17, J2 Conn_01x17, J3 Conn_01x04, U1 27C512

Commit message: fixed schottky diode part no
Parts:
- D1: value 1SS106 -> SBM245L
Changed lines of the file:
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@@
 			)
 		)
-		(property "Value" "1SS106"
+		(property "Value" "SBM245L"
 			(at 121.6025 53.34 0)
 			(effects
